File: board/DuPal_DIP/DuPal_DIP.sch (KiCad schematic (older format))
At the start: 18 parts, among them U1 ATmega8A-PU, U2 74HC595, U3 74HC595, U4 74HC595

Commit message: Add DuPal schematics changes
Parts:
- added U5: PAL16L8, symbol Logic_Programmable:PAL16L8
Connections:
- net labels added: MISO, MOSI, PAL_I1, PAL_I10, PAL_I2, PAL_I3, PAL_I4, PAL_I5, PAL_I6, PAL_I7, PAL_I8, PAL_I9, PAL_IO1, PAL_IO10, PAL_IO11, PAL_IO12, PAL_IO13, PAL_IO14, PAL_IO2, PAL_IO3, PAL_IO4, PAL_IO5, PAL_IO6, PAL_IO7, PAL_IO8, PAL_IO9, SCK, TTL-RX, TTL-TX, XTAL1, XTAL2, ~RESET
- wire segments 55 -> 94

Commit message: Add oscillator
Parts:
- added C1, C2: 22pF, symbol Device:C_Small
- added D1: LED, symbol Device:LED_Small
- added J1: AVR-ISP-6, symbol Connector:AVR-ISP-6
- added R15: 10K, symbol Device:R_Small
- added R16: 470, symbol Device:R_Small
- added R17: 1M, symbol Device:R_Small
- added SW1: SW_Push, symbol Switch:SW_Push
- added Y1: 8Mhz, symbol Device:Crystal
Connections:
- net labels added: SHFT_CLK, SHFT_RCLK, SHFT_SER, ~SHFT_OE, ~SHFT_RESET
- wire segments 94 -> 145

Commit message: More schematis changes
Parts:
- added C3: 100nF, symbol Device:C_Small
- added U6: MAX232, symbol Interface_UART:MAX232
Connections:
- net labels added: DTR, RS232-RX, RS232-TX
- wire segments 145 -> 155
Other:
- moved on the sheet: R15, R16

Commit message: Complete schematic of PAL dumper
Parts:
- removed R10, R11, R12, R13, R14, R9: 10K, symbol Device:R_Small
- removed U4: 74HC595, symbol 74xx:74HC595
- added C10, C11, C12, C14, C8, C9: 100nF, symbol Device:C_Small
- added C15: 0.22uF, symbol Device:CP1_Small
- added C4, C5, C6, C7: 1.0uF, symbol Device:CP1_Small
- added D2: LED, symbol Device:LED_Small
- added D3: 1N4001, Diode_THT:D_DO-41_SOD81_P10.16mm_Horizontal, symbol Diode:1N4001
- added J2: RS232, symbol Connector:DB9_Female_MountingHoles
- added J2: Power IN, symbol Connector:Conn_Coaxial_Power
- added R17: 1.2K, symbol Device:R_Small
- added SW2: Power, symbol Switch:SW_SPST
- added U7: L7805, symbol Regulator_Linear:L7805
Connections:
- net labels added: +12V, RECT_V12, RS232-DTR, SW_12V
- net labels removed: DTR, PAL_IO10, PAL_IO11, PAL_IO12, PAL_IO13, PAL_IO14, PAL_IO9
- wire segments 155 -> 210
Other:
- moved on the sheet: R1, R2, R3, R4, R5, R6, R7, R8

Commit message: Change wiring
Connections:
- net labels added: PAL_TRIO1, PAL_TRIO2
- net labels removed: PAL_IO7, PAL_IO8
Changed lines of the file:
@@
 PAL_IO6
 Text Label 4000 3400 2    50   ~ 0
-PAL_IO7
+PAL_TRIO1
 Text Label 4000 3500 2    50   ~ 0
-PAL_IO8
+PAL_TRIO2
+Wire Wire Line
+	7200 1250 7750 1250
+Wire Wire Line
+	7200 1350 7750 1350
+Wire Wire Line
+	7200 1450 7750 1450
+Wire Wire Line
+	7200 1550 7750 1550
+Wire Wire Line
+	7200 1650 7750 1650
+Wire Wire Line
+	7200 1750 7750 1750
 Wire Wire Line
 	7200 1150 7750 1150
 Wire Wire Line
-	7200 1250 7750 1250
-Wire Wire Line
-	7200 1350 7750 1350
-Wire Wire Line
-	7200 1450 7750 1450
-Wire Wire Line
-	7200 1550 7750 1550
-Wire Wire Line
-	7200 1650 7750 1650
-Wire Wire Line
-	7200 1750 7750 1750
-Wire Wire Line
 	7200 1850 7750 1850
+Text Label 7750 1250 2    50   ~ 0
+PAL_IO1
+Text Label 7750 1350 2    50   ~ 0
+PAL_IO2
+Text Label 7750 1450 2    50   ~ 0
+PAL_IO3
+Text Label 7750 1550 2    50   ~ 0
+PAL_IO4
+Text Label 7750 1650 2    50   ~ 0
+PAL_IO5
+Text Label 7750 1750 2    50   ~ 0
+PAL_IO6
 Text Label 7750 1150 2    50   ~ 0
-PAL_IO1
-Text Label 7750 1250 2    50   ~ 0
-PAL_IO2
-Text Label 7750 1350 2    50   ~ 0
-PAL_IO3
-Text Label 7750 1450 2    50   ~ 0
-PAL_IO4
-Text Label 7750 1550 2    50   ~ 0
-PAL_IO5
-Text Label 7750 1650 2    50   ~ 0
-PAL_IO6
-Text Label 7750 1750 2    50   ~ 0
-PAL_IO7
+PAL_TRIO1
 Text Label 7750 1850 2    50   ~ 0
-PAL_IO8
+PAL_TRIO2
 Wire Wire Line
 	6200 1150 5500 1150
@@
 PAL_IO6
 Text Label 3400 3200 2    50   ~ 0
-PAL_IO7
+PAL_TRIO1
 Text Label 3400 3300 2    50   ~ 0
-PAL_IO8
-$Comp
-L power:GND #PWR?
+PAL_TRIO2
+$Comp
+L power:GND #PWR?

Commit message: Assigned footprints
Parts:
- C1, C2: footprint (none) -> Capacitor_THT:C_Disc_D3.0mm_W2.0mm_P2.50mm
- C10, C11, C12, C14, C3, C8, C9: footprint (none) -> Capacitor_THT:C_Disc_D3.4mm_W2.1mm_P2.50mm
- C15, C4, C5, C7: footprint (none) -> Capacitor_THT:CP_Radial_D5.0mm_P2.50mm
- D1: value LED -> DATA_LED; footprint (none) -> LED_THT:LED_D2.0mm_W4.8mm_H2.5mm_FlatTop
- D2: value LED -> POWER_LED; footprint (none) -> LED_THT:LED_D2.0mm_W4.8mm_H2.5mm_FlatTop
- J1: footprint (none) -> Connector_IDC:IDC-Header_2x03_P2.54mm_Vertical
- J2: footprint (none) -> Connector_Dsub:DSUB-9_Female_Horizontal_P2.77x2.84mm_EdgePinOffset4.94mm_Housed_MountingHolesOffset7.48mm
- J2: footprint (none) -> Connector_BarrelJack:BarrelJack_Horizontal
- R1, R15, R16, R17, R2, R3, R4, R5, R6, R7, R8: footprint (none) -> Resistor_THT:R_Axial_DIN0204_L3.6mm_D1.6mm_P7.62mm_Horizontal
- SW1: footprint (none) -> Button_Switch_THT:SW_PUSH_6mm
- SW2: footprint (none) -> Button_Switch_THT:SW_Slide_1P2T_CK_OS102011MS2Q
- U2, U3: footprint (none) -> Package_DIP:DIP-16_W7.62mm
- U5: footprint (none) -> Socket:DIP_Socket-20_W4.3_W5.08_W7.62_W10.16_W10.9_3M_220-3342-00-0602J
- U6, U7: footprint (none) -> Package_TO_SOT_THT:TO-220-3_Vertical
- Y1: footprint (none) -> Crystal:Crystal_HC49-U_Vertical
Changed lines of the file:
@@
 encoding utf-8
 Sheet 1 1
-Title ""
+Title "DuPAL"
 Date ""
 Rev ""
@@
 F 0 "U2" H 9050 3150 50  0000 C CNN
 F 1 "74HC595" H 9550 3150 50  0000 C CNN
-F 2 "" H 9300 2600 50  0001 C CNN
+F 2 "Package_DIP:DIP-16_W7.62mm" H 9300 2600 50  0001 C CNN
 F 3 "http://www.ti.com/lit/ds/symlink/sn74hc595.pdf" H 9300 2600 50  0001 C CNN
 	1    9300 2600
@@
 F 0 "U3" H 9050 5050 50  0000 C CNN
 F 1 "74HC595" H 9550 5050 50  0000 C CNN
-F 2 "" H 9300 4500 50  0001 C CNN
+F 2 "Package_DIP:DIP-16_W7.62mm" H 9300 4500 50  0001 C CNN
 F 3 "http://www.ti.com/lit/ds/symlink/sn74hc595.pdf" H 9300 4500 50  0001 C CNN
 	1    9300 4500
@@
 F 0 "R1" V 10250 4450 50  0000 C CNN
 F 1 "10K" V 10250 4150 50  0000 C CNN
-F 2 "" H 10200 4300 50  0001 C CNN
+F 2 "Resistor_THT:R_Axial_DIN0204_L3.6mm_D1.6mm_P7.62mm_Horizontal" H 10200 4300 50  0001 C CNN
 F 3 "~" H 10200 4300 50  0001 C CNN
 	1    10200 4300
@@
 F 0 "R2" V 10250 4550 50  0000 C CNN
 F 1 "10K" V 10250 4250 50  0000 C CNN
-F 2 "" H 10200 4400 50  0001 C CNN
+F 2 "Resistor_THT:R_Axial_DIN0204_L3.6mm_D1.6mm_P7.62mm_Horizontal" H 10200 4400 50  0001 C CNN
 F 3 "~" H 10200 4400 50  0001 C CNN
 	1    10200 4400
@@
 F 0 "R3" V 10250 4650 50  0000 C CNN
 F 1 "10K" V 10250 4350 50  0000 C CNN
-F 2 "" H 10200 4500 50  0001 C CNN
+F 2 "Resistor_THT:R_Axial_DIN0204_L3.6mm_D1.6mm_P7.62mm_Horizontal" H 10200 4500 50  0001 C CNN
 F 3 "~" H 10200 4500 50  0001 C CNN
 	1    10200 4500
@@
 F 0 "R4" V 10250 4750 50  0000 C CNN
 F 1 "10K" V 10250 4450 50  0000 C CNN
-F 2 "" H 10200 4600 50  0001 C CNN
+F 2 "Resistor_THT:R_Axial_DIN0204_L3.6mm_D1.6mm_P7.62mm_Horizontal" H 10200 4600 50  0001 C CNN
 F 3 "~" H 10200 4600 50  0001 C CNN
 	1    10200 4600
@@
 F 0 "R5" V 10250 4850 50  0000 C CNN
 F 1 "10K" V 10250 4550 50  0000 C CNN
-F 2 "" H 10200 4700 50  0001 C CNN
+F 2 "Resistor_THT:R_Axial_DIN0204_L3.6mm_D1.6mm_P7.62mm_Horizontal" H 10200 4700 50  0001 C CNN
 F 3 "~" H 10200 4700 50  0001 C CNN
 	1    10200 4700
@@
 F 0 "R6" V 10250 4950 50  0000 C CNN
 F 1 "10K" V 10250 4650 50  0000 C CNN
-F 2 "" H 10200 4800 50  0001 C CNN
+F 2 "Resistor_THT:R_Axial_DIN0204_L3.6mm_D1.6mm_P7.62mm_Horizontal" H 10200 4800 50  0001 C CNN
 F 3 "~" H 10200 4800 50  0001 C CNN
 	1    10200 4800
@@
 F 0 "R7" V 3450 3550 50  0000 C CNN
 F 1 "10K" V 3450 3250 50  0000 C CNN
-F 2 "" H 3400 3400 50  0001 C CNN
+F 2 "Resistor_THT:R_Axial_DIN0204_L3.6mm_D1.6mm_P7.62mm_Horizontal" H 3400 3400 50  0001 C CNN
 F 3 "~" H 3400 3400 50  0001 C CNN
 	1    3400 3400
@@
 F 0 "R8" V 3450 3650 50  0000 C CNN
 F 1 "10K" V 3450 3350 50  0000 C CNN
-F 2 "" H 3400 3500 50  0001 C CNN
+F 2 "Resistor_THT:R_Axial_DIN0204_L3.6mm_D1.6mm_P7.62mm_Horizontal" H 3400 3500 50  0001 C CNN
 F 3 "~" H 3400 3500 50  0001 C CNN
 	1    3400 3500
@@
 F 0 "U5" H 6400 2250 50  0000 C CNN
 F 1 "PAL16L8" H 6950 2250 50  0000 C CNN
-F 2 "" H 6700 1650 50  0001 C CNN
+F 2 "Socket:DIP_Socket-20_W4.3_W5.08_W7.62_W10.16_W10.9_3M_220-3342-00-0602J" H 6700 1650 50  0001 C CNN
 F 3 "" H 6700 1650 50  0001 C CNN
 	1    6700 1650
@@
 F 0 "R15" V 1296 1400 50  0000 C CNN
 F 1 "10K" V 1205 1400 50  0000 C CNN
-F 2 "" H 1100 1400 50  0001 C CNN
+F 2 "Resistor_THT:R_Axial_DIN0204_L3.6mm_D1.6mm_P7.62mm_Horizontal" H 1100 1400 50  0001 C CNN
 F 3 "~" H 1100 1400 50  0001 C CNN
 	1    1100 1400
@@
 F 0 "J1" H 6471 3496 50  0000 R CNN
 F 1 "AVR-ISP-6" H 6471 3405 50  0000 R CNN
-F 2 "" V 6550 3450 50  0001 C CNN
+F 2 "Connector_IDC:IDC-Header_2x03_P2.54mm_Vertical" V 6550 3450 50  0001 C CNN
 F 3 " ~" H 5525 2850 50  0001 C CNN
 	1    6800 3400
@@
 F 0 "SW1" H 7500 4000 50  0000 C CNN
 F 1 "SW_Push" H 7500 3700 50  0000 C CNN
-F 2 "" H 7500 4000 50  0001 C CNN
+F 2 "Button_Switch_THT:SW_PUSH_6mm" H 7500 4000 50  0001 C CNN
 F 3 "~" H 7500 4000 50  0001 C CNN
 	1    7500 3800
@@
 P 3650 1900
 F 0 "D1" H 3650 2135 50  0000 C CNN
-F 1 "LED" H 3650 2044 50  0000 C CNN
-F 2 "" V 3650 1900 50  0001 C CNN
+F 1 "DATA_LED" H 3650 2044 50  0000 C CNN
+F 2 "LED_THT:LED_D2.0mm_W4.8mm_H2.5mm_FlatTop" V 3650 1900 50  0001 C CNN
 F 3 "~" V 3650 1900 50  0001 C CNN
 	1    3650 1900
@@
 F 0 "R16" V 4146 1900 50  0000 C CNN
 F 1 "470" V 4055 1900 50  0000 C CNN
-F 2 "" H 3950 1900 50  0001 C CNN
+F 2 "Resistor_THT:R_Axial_DIN0204_L3.6mm_D1.6mm_P7.62mm_Horizontal" H 3950 1900 50  0001 C CNN
 F 3 "~" H 3950 1900 50  0001 C CNN
 	1    3950 1900
@@
 F 0 "Y1" V 7100 4800 50  0000 R CNN
 F 1 "8Mhz" V 7000 4900 50  0000 R CNN
-F 2 "" H 7050 4600 50  0001 C CNN
+F 2 "Crystal:Crystal_HC49-U_Vertical" H 7050 4600 50  0001 C CNN
 F 3 "~" H 7050 4600 50  0001 C CNN
 	1    7050 4600
@@
 F 0 "C1" V 6829 4450 50  0000 C CNN
 F 1 "22pF" V 6738 4450 50  0000 C CNN
-F 2 "" H 6600 4450 50  0001 C CNN
+F 2 "Capacitor_THT:C_Disc_D3.0mm_W2.0mm_P2.50mm" H 6600 4450 50  0001 C CNN
 F 3 "~" H 6600 4450 50  0001 C CNN
 	1    6600 4450
@@
 F 0 "C2" V 6450 4750 50  0000 C CNN
 F 1 "22pF" V 6738 4750 50  0000 C CNN
-F 2 "" H 6600 4750 50  0001 C CNN
+F 2 "Capacitor_THT:C_Disc_D3.0mm_W2.0mm_P2.50mm" H 6600 4750 50  0001 C CNN
 F 3 "~" H 6600 4750 50  0001 C CNN
 	1    6600 4750
@@
 F 0 "U6" H 1800 7200 50  0000 C CNN
 F 1 "MAX232" H 2800 7200 50  0000 C CNN
-F 2 "" H 2400 5050 50  0001 L CNN
+F 2 "Package_TO_SOT_THT:TO-220-3_Vertical" H 2400 5050 50  0001 L CNN
 F 3 "http://www.ti.com/lit/ds/symlink/max232.pdf" H 2350 6200 50  0001 C CNN
 	1    2350 6100
@@
 F 0 "C3" V 1350 6700 50  0000 C CNN
 F 1 "100nF" V 1350 6450 50  0000 C CNN
-F 2 "" H 1300 6600 50  0001 C CNN
+F 2 "Capacitor_THT:C_Disc_D3.4mm_W2.1mm_P2.50mm" H 1300 6600 50  0001 C CNN
 F 3 "~" H 1300 6600 50  0001 C CNN
 	1    1300 6600
@@
 F 0 "C4" H 1441 5396 50  0000 L CNN
 F 1 "1.0uF" H 1441 5305 50  0000 L CNN
-F 2 "" H 1350 5350 50  0001 C CNN
+F 2 "Capacitor_THT:CP_Radial_D5.0mm_P2.50mm" H 1350 5350 50  0001 C CNN
 F 3 "~" H 1350 5350 50  0001 C CNN
 	1    1350 5350
@@
 F 0 "C5" H 3391 5396 50  0000 L CNN
 F 1 "1.0uF" H 3391 5305 50  0000 L CNN
-F 2 "" H 3300 5350 50  0001 C CNN
+F 2 "Capacitor_THT:CP_Radial_D5.0mm_P2.50mm" H 3300 5350 50  0001 C CNN
 F 3 "~" H 3300 5350 50  0001 C CNN
 	1    3300 5350
@@
 F 0 "C7" V 3750 6000 50  0000 C CNN
 F 1 "1.0uF" V 3513 6000 50  0000 C CNN
-F 2 "" H 3650 6000 50  0001 C CNN
+F 2 "Capacitor_THT:CP_Radial_D5.0mm_P2.50mm" H 3650 6000 50  0001 C CNN
 F 3 "~" H 3650 6000 50  0001 C CNN
 	1    3650 6000
@@
 F 0 "J2" H 7230 5652 50  0000 L CNN
 F 1 "RS232" H 7230 5561 50  0000 L CNN
-F 2 "" H 7050 5650 50  0001 C CNN
+F 2 "Connector_Dsub:DSUB-9_Female_Horizontal_P2.77x2.84mm_EdgePinOffset4.94mm_Housed_MountingHolesOffset7.48mm" H 7050 5650 50  0001 C CNN
 F 3 " ~" H 7050 5650 50  0001 C CNN
 	1    7050 5650
@@
 F 0 "C8" V 5000 2750 50  0000 C CNN
 F 1 "100nF" V 5000 2450 50  0000 C CNN
-F 2 "" H 4950 2600 50  0001 C CNN
+F 2 "Capacitor_THT:C_Disc_D3.4mm_W2.1mm_P2.50mm" H 4950 2600 50  0001 C CNN
 F 3 "~" H 4950 2600 50  0001 C CNN
 	1    4950 2600
@@
 F 0 "C9" V 5000 2950 50  0000 C CNN
 F 1 "100nF" V 5000 2650 50  0000 C CNN
-F 2 "" H 4950 2800 50  0001 C CNN
+F 2 "Capacitor_THT:C_Disc_D3.4mm_W2.1mm_P2.50mm" H 4950 2800 50  0001 C CNN
 F 3 "~" H 4950 2800 50  0001 C CNN
 	1    4950 2800
@@
 F 0 "C10" V 5000 3150 50  0000 C CNN
 F 1 "100nF" V 5000 2850 50  0000 C CNN
-F 2 "" H 4950 3000 50  0001 C CNN
+F 2 "Capacitor_THT:C_Disc_D3.4mm_W2.1mm_P2.50mm" H 4950 3000 50  0001 C CNN
 F 3 "~" H 4950 3000 50  0001 C CNN
 	1    4950 3000
@@
 F 0 "C11" V 5000 3350 50  0000 C CNN
 F 1 "100nF" V 5000 3050 50  0000 C CNN
-F 2 "" H 4950 3200 50  0001 C CNN
+F 2 "Capacitor_THT:C_Disc_D3.4mm_W2.1mm_P2.50mm" H 4950 3200 50  0001 C CNN
 F 3 "~" H 4950 3200 50  0001 C CNN
 	1    4950 3200
@@
 F 0 "C12" V 5000 3550 50  0000 C CNN
 F 1 "100nF" V 5000 3250 50  0000 C CNN
-F 2 "" H 4950 3400 50  0001 C CNN
+F 2 "Capacitor_THT:C_Disc_D3.4mm_W2.1mm_P2.50mm" H 4950 3400 50  0001 C CNN
 F 3 "~" H 4950 3400 50  0001 C CNN
 	1    4950 3400
@@
 F 0 "U7" H 5000 4742 50  0000 C CNN
 F 1 "L7805" H 5000 4651 50  0000 C CNN
-F 2 "" H 5025 4350 50  0001 L CIN
+F 2 "Package_TO_SOT_THT:TO-220-3_Vertical" H 5025 4350 50  0001 L CIN
 F 3 "http://www.st.com/content/ccc/resource/technical/document/datasheet/41/4f/b3/b0/12/d4/47/88/CD00000444.pdf/files/CD00000444.pdf/jcr:content/translations/en.CD00000444.pdf" H 5000 4450 50  0001 C CNN
 	1    5000 4500
@@
 F 0 "C14" H 5600 4800 50  0000 C CNN
 F 1 "100nF" H 5650 4600 50  0000 C CNN
-F 2 "" H 5500 4700 50  0001 C CNN
+F 2 "Capacitor_THT:C_Disc_D3.4mm_W2.1mm_P2.50mm" H 5500 4700 50  0001 C CNN
 F 3 "~" H 5500 4700 50  0001 C CNN
 	1    5500 4700
@@
 F 0 "C15" H 4591 4746 50  0000 L CNN
 F 1 "0.22uF" H 4591 4655 50  0000 L CNN
-F 2 "" H 4500 4700 50  0001 C CNN
+F 2 "Capacitor_THT:CP_Radial_D5.0mm_P2.50mm" H 4500 4700 50  0001 C CNN
 F 3 "~" H 4500 4700 50  0001 C CNN
 	1    4500 4700
@@
 P 4850 5500
 F 0 "D2" H 4850 5735 50  0000 C CNN
-F 1 "LED" H 4850 5644 50  0000 C CNN
-F 2 "" V 4850 5500 50  0001 C CNN
+F 1 "POWER_LED" H 4850 5644 50  0000 C CNN
+F 2 "LED_THT:LED_D2.0mm_W4.8mm_H2.5mm_FlatTop" V 4850 5500 50  0001 C CNN
 F 3 "~" V 4850 5500 50  0001 C CNN
 	1    4850 5500
@@
 F 0 "R17" V 5346 5500 50  0000 C CNN
 F 1 "1.2K" V 5255 5500 50  0000 C CNN
-F 2 "" H 5150 5500 50  0001 C CNN
+F 2 "Resistor_THT:R_Axial_DIN0204_L3.6mm_D1.6mm_P7.62mm_Horizontal" H 5150 5500 50  0001 C CNN
 F 3 "~" H 5150 5500 50  0001 C CNN
 	1    5150 5500
@@
 F 0 "SW2" H 4650 6285 50  0000 C CNN
 F 1 "Power" H 4650 6194 50  0000 C CNN
-F 2 "" H 4650 6050 50  0001 C CNN
+F 2 "Button_Switch_THT:SW_Slide_1P2T_CK_OS102011MS2Q" H 4650 6050 50  0001 C CNN
 F 3 "~" H 4650 6050 50  0001 C CNN
 	1    4650 6050
@@
 F 0 "J2" V 4733 6550 50  0000 C CNN
 F 1 "Power IN" V 4824 6550 50  0000 C CNN
-F 2 "" H 4950 6550 50  0001 C CNN
+F 2 "Connector_BarrelJack:BarrelJack_Horizontal" H 4950 6550 50  0001 C CNN
 F 3 "~" H 4950 6550 50  0001 C CNN
 	1    4950 6600

Commit message: Add correct footprints
Parts:
- C6: footprint (none) -> Capacitor_THT:CP_Radial_D5.0mm_P2.50mm
- R18: renamed from R17; footprint (none) -> Resistor_THT:R_Axial_DIN0204_L3.6mm_D1.6mm_P7.62mm_Horizontal
- U6: footprint Package_TO_SOT_THT:TO-220-3_Vertical -> Package_DIP:DIP-16_W7.62mm
- renumbered J2 to J3
Changed lines of the file:
@@
 $EndComp
 $Comp
-L power:VCC #PWR?
+L power:VCC #PWR0101
 U 1 1 5E54FA95
 P 9300 1950
-F 0 "#PWR?" H 9300 1800 50  0001 C CNN
+F 0 "#PWR0101" H 9300 1800 50  0001 C CNN
 F 1 "VCC" H 9317 2123 50  0000 C CNN
 F 2 "" H 9300 1950 50  0001 C CNN
@@
 	9300 1950 9300 2000
 $Comp
-L power:VCC #PWR?
+L power:VCC #PWR0102
 U 1 1 5E5508CD
 P 9300 3850
-F 0 "#PWR?" H 9300 3700 50  0001 C CNN
+F 0 "#PWR0102" H 9300 3700 50  0001 C CNN
 F 1 "VCC" H 9317 4023 50  0000 C CNN
 F 2 "" H 9300 3850 50  0001 C CNN
@@
 	9300 5200 9300 5250
 $Comp
-L power:GND #PWR?
+L power:GND #PWR0103
 U 1 1 5E55166F
 P 9300 3350
-F 0 "#PWR?" H 9300 3100 50  0001 C CNN
+F 0 "#PWR0103" H 9300 3100 50  0001 C CNN
 F 1 "GND" H 9305 3177 50  0000 C CNN
 F 2 "" H 9300 3350 50  0001 C CNN
@@
 $EndComp
 $Comp
-L power:GND #PWR?
+L power:GND #PWR0104
 U 1 1 5E551F7F
 P 6700 2300
-F 0 "#PWR?" H 6700 2050 50  0001 C CNN
+F 0 "#PWR0104" H 6700 2050 50  0001 C CNN
 F 1 "GND" H 6705 2127 50  0000 C CNN
 F 2 "" H 6700 2300 50  0001 C CNN
@@
 	6700 2300 6700 2250
 $Comp
-L power:VCC #PWR?
+L power:VCC #PWR0105
 U 1 1 5E5538C6
 P 6700 900
-F 0 "#PWR?" H 6700 750 50  0001 C CNN
+F 0 "#PWR0105" H 6700 750 50  0001 C CNN
 F 1 "VCC" H 6717 1073 50  0000 C CNN
 F 2 "" H 6700 900 50  0001 C CNN
@@
 PAL_I10
 $Comp
-L power:VCC #PWR?
+L power:VCC #PWR0106
 U 1 1 5E5B3D6B
 P 2350 900
-F 0 "#PWR?" H 2350 750 50  0001 C CNN
+F 0 "#PWR0106" H 2350 750 50  0001 C CNN
 F 1 "VCC" H 2367 1073 50  0000 C CNN
 F 2 "" H 2350 900 50  0001 C CNN
@@
 	2350 1000 2400 1000
 $Comp
-L power:VCC #PWR?
+L power:VCC #PWR0107
 U 1 1 5E5BA9B3
 P 1550 2000
-F 0 "#PWR?" H 1550 1850 50  0001 C CNN
+F 0 "#PWR0107" H 1550 1850 50  0001 C CNN
 F 1 "VCC" V 1568 2127 50  0000 L CNN
 F 2 "" H 1550 2000 50  0001 C CNN
@@
 	1700 2000 1550 2000
 $Comp
-L power:GND #PWR?
+L power:GND #PWR0108
 U 1 1 5E5C11F5
 P 2350 4050
-F 0 "#PWR?" H 2350 3800 50  0001 C CNN
+F 0 "#PWR0108" H 2350 3800 50  0001 C CNN
 F 1 "GND" H 2355 3877 50  0000 C CNN
 F 2 "" H 2350 4050 50  0001 C CNN
@@
 $EndComp
 $Comp
-L power:VCC #PWR?
+L power:VCC #PWR0109
 U 1 1 5E55EA3E
 P 850 1300
-F 0 "#PWR?" H 850 1150 50  0001 C CNN
+F 0 "#PWR0109" H 850 1150 50  0001 C CNN
 F 1 "VCC" H 867 1473 50  0000 C CNN
 F 2 "" H 850 1300 50  0001 C CNN
@@
 $EndComp
 $Comp
-L power:VCC #PWR?
+L power:VCC #PWR0110
 U 1 1 5E564035
 P 6700 2850
-F 0 "#PWR?" H 6700 2700 50  0001 C CNN
+F 0 "#PWR0110" H 6700 2700 50  0001 C CNN
 F 1 "VCC" H 6717 3023 50  0000 C CNN
 F 2 "" H 6700 2850 50  0001 C CNN
@@
 	6700 2850 6700 2900
 $Comp
-L power:GND #PWR?
+L power:GND #PWR0111
 U 1 1 5E5686ED
 P 6700 3850
-F 0 "#PWR?" H 6700 3600 50  0001 C CNN
+F 0 "#PWR0111" H 6700 3600 50  0001 C CNN
 F 1 "GND" H 6705 3677 50  0000 C CNN
 F 2 "" H 6700 3850 50  0001 C CNN
@@
 	3850 1900 3750 1900
 $Comp
-L power:GND #PWR?
+L power:GND #PWR0112
 U 1 1 5E61E776
 P 4150 1950
-F 0 "#PWR?" H 4150 1700 50  0001 C CNN
+F 0 "#PWR0112" H 4150 1700 50  0001 C CNN
 F 1 "GND" H 4155 1777 50  0000 C CNN
 F 2 "" H 4150 1950 50  0001 C CNN
@@
 	4050 1900 4150 1900
 $Comp
-L Device:R_Small R17
+L Device:R_Small R18
 U 1 1 5E62742F
 P 7250 4600
-F 0 "R17" H 7191 4554 50  0000 R CNN
+F 0 "R18" H 7191 4554 50  0000 R CNN
 F 1 "1M" H 7191 4645 50  0000 R CNN
-F 2 "" H 7250 4600 50  0001 C CNN
+F 2 "Resistor_THT:R_Axial_DIN0204_L3.6mm_D1.6mm_P7.62mm_Horizontal" H 7250 4600 50  0001 C CNN
 F 3 "~" H 7250 4600 50  0001 C CNN
 	1    7250 4600
@@
 $EndComp
 $Comp
-L power:GND #PWR?
+L power:GND #PWR0113
 U 1 1 5E6404B8
 P 6350 4600
-F 0 "#PWR?" H 6350 4350 50  0001 C CNN
+F 0 "#PWR0113" H 6350 4350 50  0001 C CNN
 F 1 "GND" V 6355 4472 50  0000 R CNN
 F 2 "" H 6350 4600 50  0001 C CNN
@@
 F 0 "U6" H 1800 7200 50  0000 C CNN
 F 1 "MAX232" H 2800 7200 50  0000 C CNN
-F 2 "Package_TO_SOT_THT:TO-220-3_Vertical" H 2400 5050 50  0001 L CNN
+F 2 "Package_DIP:DIP-16_W7.62mm" H 2400 5050 50  0001 L CNN
 F 3 "http://www.ti.com/lit/ds/symlink/max232.pdf" H 2350 6200 50  0001 C CNN
 	1    2350 6100
@@
 RS232-RX
 $Comp
-L power:GND #PWR?
+L power:GND #PWR0114
 U 1 1 5E6FAD32
 P 1350 6200
-F 0 "#PWR?" H 1350 5950 50  0001 C CNN
+F 0 "#PWR0114" H 1350 5950 50  0001 C CNN
 F 1 "GND" V 1355 6072 50  0000 R CNN
 F 2 "" H 1350 6200 50  0001 C CNN
@@
 	1350 6200 1550 6200
 $Comp
-L power:GND #PWR?
+L power:GND #PWR0115
 U 1 1 5E70E96E
 P 2350 7400
-F 0 "#PWR?" H 2350 7150 50  0001 C CNN
+F 0 "#PWR0115" H 2350 7150 50  0001 C CNN
 F 1 "GND" H 2355 7227 50  0000 C CNN
 F 2 "" H 2350 7400 50  0001 C CNN
@@
 	2350 7300 2350 7350
 $Comp
-L power:VCC #PWR?
+L power:VCC #PWR0116
 U 1 1 5E718EEA
 P 2350 4800
-F 0 "#PWR?" H 2350 4650 50  0001 C CNN
+F 0 "#PWR0116" H 2350 4650 50  0001 C CNN
 F 1 "VCC" H 2367 4973 50  0000 C CNN
 F 2 "" H 2350 4800 50  0001 C CNN
@@
 F 0 "C6" V 3878 5700 50  0000 C CNN
 F 1 "1.0uF" V 3787 5700 50  0000 C CNN
-F 2 "" H 3650 5700 50  0001 C CNN
+F 2 "Capacitor_THT:CP_Radial_D5.0mm_P2.50mm" H 3650 5700 50  0001 C CNN
 F 3 "~" H 3650 5700 50  0001 C CNN
 	1    3650 5700
@@
 $EndComp
 $Comp
-L power:GND #PWR?
+L power:GND #PWR0117
 U 1 1 5E796D19
 P 7300 6250
-F 0 "#PWR?" H 7300 6000 50  0001 C CNN
+F 0 "#PWR0117" H 7300 6000 50  0001 C CNN
 F 1 "GND" V 7305 6122 50  0000 R CNN
 F 2 "" H 7300 6250 50  0001 C CNN
@@
 	5250 2800 5250 3000
 $Comp
-L power:VCC #PWR?
+L power:VCC #PWR0118
 U 1 1 5E8AF29A
 P 4650 2300
-F 0 "#PWR?" H 4650 2150 50  0001 C CNN
+F 0 "#PWR0118" H 4650 2150 50  0001 C CNN
 F 1 "VCC" H 4667 2473 50  0000 C CNN
 F 2 "" H 4650 2300 50  0001 C CNN
@@
 $EndComp
 $Comp
-L power:GND #PWR?
+L power:GND #PWR0119
 U 1 1 5E8AF8D2
 P 5250 3850
-F 0 "#PWR?" H 5250 3600 50  0001 C CNN
+F 0 "#PWR0119" H 5250 3600 50  0001 C CNN
 F 1 "GND" H 5255 3677 50  0000 C CNN
 F 2 "" H 5250 3850 50  0001 C CNN
@@
 $EndComp
 $Comp
-L power:GND #PWR?
+L power:GND #PWR0120
 U 1 1 5E8C0D79
 P 5000 5000
-F 0 "#PWR?" H 5000 4750 50  0001 C CNN
+F 0 "#PWR0120" H 5000 4750 50  0001 C CNN
 F 1 "GND" H 5005 4827 50  0000 C CNN
 F 2 "" H 5000 5000 50  0001 C CNN
@@
 Connection ~ 5500 4500
 $Comp
-L power:VCC #PWR?
+L power:VCC #PWR0121
 U 1 1 5E91370A
 P 5500 4300
-F 0 "#PWR?" H 5500 4150 50  0001 C CNN
+F 0 "#PWR0121" H 5500 4150 50  0001 C CNN
 F 1 "VCC" H 5517 4473 50  0000 C CNN
 F 2 "" H 5500 4300 50  0001 C CNN
@@
 	5050 5500 4950 5500
 $Comp
-L power:GND #PWR?
+L power:GND #PWR0122
 U 1 1 5E98E821
 P 5500 5550
-F 0 "#PWR?" H 5500 5300 50  0001 C CNN
+F 0 "#PWR0122" H 5500 5300 50  0001 C CNN
 F 1 "GND" H 5505 5377 50  0000 C CNN
 F 2 "" H 5500 5550 50  0001 C CNN
@@
 $EndComp
 $Comp
-L Connector:Conn_Coaxial_Power J2
+L Connector:Conn_Coaxial_Power J3
 U 1 1 5E9B6738
 P 4950 6600
-F 0 "J2" V 4733 6550 50  0000 C CNN
+F 0 "J3" V 4733 6550 50  0000 C CNN
 F 1 "Power IN" V 4824 6550 50  0000 C CNN
 F 2 "Connector_BarrelJack:BarrelJack_Horizontal" H 4950 6550 50  0001 C CNN
@@
 $EndComp
 $Comp
-L power:GND #PWR?
+L power:GND #PWR0123
 U 1 1 5E9C89CF
 P 4650 6700
-F 0 "#PWR?" H 4650 6450 50  0001 C CNN
+F 0 "#PWR0123" H 4650 6450 50  0001 C CNN
 F 1 "GND" H 4655 6527 50  0000 C CNN
 F 2 "" H 4650 6700 50  0001 C CNN
@@
 	4650 6600 4750 6600
 $Comp
-L power:+12V #PWR?
+L power:+12V #PWR0124
 U 1 1 5E9DAF23
 P 5150 6700
-F 0 "#PWR?" H 5150 6550 50  0001 C CNN
+F 0 "#PWR0124" H 5150 6550 50  0001 C CNN
 F 1 "+12V" H 5165 6873 50  0000 C CNN
 F 2 "" H 5150 6700 50  0001 C CNN
@@
 	5150 6600 5150 6700
 $Comp
-L power:+12V #PWR?
+L power:+12V #PWR0125
 U 1 1 5EA26609
 P 4350 5950
-F 0 "#PWR?" H 4350 5800 50  0001 C CNN
+F 0 "#PWR0125" H 4350 5800 50  0001 C CNN
 F 1 "+12V" H 4365 6123 50  0000 C CNN
 F 2 "" H 4350 5950 50  0001 C CNN
@@
 PAL_TRIO2
 $Comp
-L power:GND #PWR?
+L power:GND #PWR0126
 U 1 1 5E550F46
 P 9300 5250
-F 0 "#PWR?" H 9300 5000 50  0001 C CNN
+F 0 "#PWR0126" H 9300 5000 50  0001 C CNN
 F 1 "GND" H 9305 5077 50  0000 C CNN
 F 2 "" H 9300 5250 50  0001 C CNN
