File: board/DuPal_DIP/DuPal_DIP.sch (KiCad schematic (older format))
At the start: 41 parts, among them J1 AVR-ISP-6, J2 RS232, J3 Power IN, SW1 SW_Push, SW2 Power, U1 ATmega8A-PU, U2 74HC595, U3 74HC595, U5 PAL16L8, U6 MAX232, U7 L7805, Y1 8Mhz

Commit message: Begin adding new shift and parallel registers
Parts:
- added U? (x2): 74HC595, Package_DIP:DIP-16_W7.62mm, symbol 74xx:74HC595
- added U? (x2): 74HC166, symbol 74xx_IEEE:74166
Connections:
- net labels added: PISO_CLK, PISO_INH, PISO_SER, PISO_SH, SIPO_CLK, SIPO_RCLK, SIPO_SER, ~PISO_CLR, ~SIPO_CLR, ~SIPO_OE
- net labels removed: SHFT_CLK, SHFT_RCLK, SHFT_SER, ~SHFT_OE, ~SHFT_RESET
- wire segments 210 -> 303
Other:
- moved on the sheet: R1, R2, R3, R4, R5, R6
