File: board/DuPal_DIP/DuPal_DIP.sch (KiCad schematic (older format))
At the start: 45 parts, among them J1 AVR-ISP-6, J2 RS232, J3 Power IN, SW1 SW_Push, SW2 Power, U1 ATmega8A-PU, U2 74HC595, U3 74HC595, U5 PAL16L8, U6 MAX232, U7 L7805, Y1 8Mhz

Commit message: Begin remapping the connections
Parts:
- removed U?: 74HC595, Package_DIP:DIP-16_W7.62mm, symbol 74xx:74HC595
- added U?: FT232RL, Package_SO:SSOP-28_5.3x10.2mm_P0.65mm, symbol Interface_USB:FT232RL
- U5: value PAL16L8 -> 20 Pin PAL
Connections:
- net labels added: P20_1, P20_11, P20_12, P20_13, P20_14, P20_15, P20_16, P20_17, P20_18, P20_19, P20_2, P20_3, P20_4, P20_5, P20_6, P20_7, P20_8, P20_9, SIPO_O_1, SIPO_O_10, SIPO_O_11, SIPO_O_12, SIPO_O_13, SIPO_O_14, SIPO_O_15, SIPO_O_16, SIPO_O_17, SIPO_O_18, SIPO_O_19, SIPO_O_2, SIPO_O_20, SIPO_O_21, SIPO_O_22, SIPO_O_23, SIPO_O_24, SIPO_O_3, SIPO_O_4, SIPO_O_5, SIPO_O_6, SIPO_O_7, SIPO_O_8, SIPO_O_9
- net labels removed: PAL_I1, PAL_I10, PAL_I2, PAL_I3, PAL_I4, PAL_I5, PAL_I6, PAL_I7, PAL_I8, PAL_I9, PAL_IO1, PAL_IO2, PAL_IO3, PAL_IO4, PAL_IO5, PAL_IO6, PAL_TRIO1, PAL_TRIO2
- wire segments 303 -> 298
Other:
- moved on the sheet: R1, R2, R3, R4, R5, R6, R7, R8
