File: board/DuPal_DIP/DuPal_DIP.sch (KiCad schematic (older format))
At the start: 55 parts, among them J1 AVR-ISP-6, J2 RS232, J3 Power IN, SW1 SW_Push, SW2 Power, U1 ATmega8A-PU, U10 24 Pin PAL, U2 74HC595, U3 74HC595, U5 20 Pin PAL, U6 MAX232, U7 74HC595, U7 L7805, U8 74HC166, Y1 8Mhz

Commit message: Begin reworking the PCB
Parts:
- U7: footprint Package_TO_SOT_THT:TO-220-3_Vertical -> Package_TO_SOT_THT:TO-220-3_Horizontal_TabDown
- renumbered C14 to C16, C15 to C17, U7 to U9
Changed lines of the file:
@@
 F 0 "U7" H 5000 4742 50  0000 C CNN
 F 1 "L7805" H 5000 4651 50  0000 C CNN
-F 2 "Package_TO_SOT_THT:TO-220-3_Vertical" H 5025 4350 50  0001 L CIN
+F 2 "Package_TO_SOT_THT:TO-220-3_Horizontal_TabDown" H 5025 4350 50  0001 L CIN
 F 3 "http://www.st.com/content/ccc/resource/technical/document/datasheet/41/4f/b3/b0/12/d4/47/88/CD00000444.pdf/files/CD00000444.pdf/jcr:content/translations/en.CD00000444.pdf" H 5000 4450 50  0001 C CNN
 	1    5000 4500
@@
 	4300 5500 4750 5500
 $Comp
-L 74xx:74HC595 U7
+L 74xx:74HC595 U9
 U 1 1 5F3CD878
 P 13850 5300
-F 0 "U7" H 13600 5850 50  0000 C CNN
+F 0 "U9" H 13600 5850 50  0000 C CNN
 F 1 "74HC595" H 14100 5850 50  0000 C CNN
 F 2 "Package_DIP:DIP-16_W7.62mm" H 13850 5300 50  0001 C CNN
@@
 $EndComp
 $Comp
-L Device:C_Small C14
+L Device:C_Small C16
 U 1 1 619A5323
 P 1750 9750
-F 0 "C14" V 1800 9900 50  0000 C CNN
+F 0 "C16" V 1800 9900 50  0000 C CNN
 F 1 "100nF" V 1800 9600 50  0000 C CNN
 F 2 "Capacitor_THT:C_Disc_D3.4mm_W2.1mm_P2.50mm" H 1750 9750 50  0001 C CNN
@@
 	1850 9750 2050 9750
 $Comp
-L Device:C_Small C15
+L Device:C_Small C17
 U 1 1 61A81BD7
 P 1750 9950
-F 0 "C15" V 1800 10100 50  0000 C CNN
+F 0 "C17" V 1800 10100 50  0000 C CNN
 F 1 "100nF" V 1800 9800 50  0000 C CNN
 F 2 "Capacitor_THT:C_Disc_D3.4mm_W2.1mm_P2.50mm" H 1750 9950 50  0001 C CNN

Commit message: First PCB model for Rev.2
Parts:
- H1, H2, H3, H4: footprint (none) -> MountingHole:MountingHole_2.7mm_M2.5_ISO7380_Pad
Changed lines of the file:
@@
 F 0 "H1" H 5750 8649 50  0000 L CNN
 F 1 "MountingHole_Pad" H 5750 8558 50  0000 L CNN
-F 2 "" H 5650 8600 50  0001 C CNN
+F 2 "MountingHole:MountingHole_2.7mm_M2.5_ISO7380_Pad" H 5650 8600 50  0001 C CNN
 F 3 "~" H 5650 8600 50  0001 C CNN
 	1    5650 8600
@@
 F 0 "H2" H 6900 8649 50  0000 L CNN
 F 1 "MountingHole_Pad" H 6900 8558 50  0000 L CNN
-F 2 "" H 6800 8600 50  0001 C CNN
+F 2 "MountingHole:MountingHole_2.7mm_M2.5_ISO7380_Pad" H 6800 8600 50  0001 C CNN
 F 3 "~" H 6800 8600 50  0001 C CNN
 	1    6800 8600
@@
 F 0 "H3" H 5750 9449 50  0000 L CNN
 F 1 "MountingHole_Pad" H 5750 9358 50  0000 L CNN
-F 2 "" H 5650 9400 50  0001 C CNN
+F 2 "MountingHole:MountingHole_2.7mm_M2.5_ISO7380_Pad" H 5650 9400 50  0001 C CNN
 F 3 "~" H 5650 9400 50  0001 C CNN
 	1    5650 9400
@@
 F 0 "H4" H 6900 9449 50  0000 L CNN
 F 1 "MountingHole_Pad" H 6900 9358 50  0000 L CNN
-F 2 "" H 6800 9400 50  0001 C CNN
+F 2 "MountingHole:MountingHole_2.7mm_M2.5_ISO7380_Pad" H 6800 9400 50  0001 C CNN
 F 3 "~" H 6800 9400 50  0001 C CNN
 	1    6800 9400
