File: board/dupico_pods/pod_pal/pod_pal.kicad_sch (KiCad schematic)
At the start: 8 parts, among them J1 dupico, J2 GAL, Q1 2N3906, U1 74HCT04

Commit message: Update pal pod for dupico
Parts:
- R1: value 2.2k -> 1k
- U1: value 74HCT04 -> 74ACT04
Changed lines of the file:
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@@
 			)
 		)
-		(property "Value" "74HCT04"
+		(property "Value" "74ACT04"
 			(at 247.65 149.86 0)
 			(effects
@@
 			)
 		)
-		(property "Value" "74HCT04"
+		(property "Value" "74ACT04"
 			(at 247.65 107.95 0)
 			(effects
@@
 			)
 		)
-		(property "Value" "74HCT04"
+		(property "Value" "74ACT04"
 			(at 247.65 135.89 0)
 			(effects
@@
 			)
 		)
-		(property "Value" "74HCT04"
+		(property "Value" "74ACT04"
 			(at 250.19 50.7999 0)
 			(effects
@@
 			)
 		)
-		(property "Value" "74HCT04"
+		(property "Value" "74ACT04"
 			(at 134.62 110.49 0)
 			(effects
@@
 			)
 		)
-		(property "Value" "74HCT04"
+		(property "Value" "74ACT04"
 			(at 247.65 93.98 0)
 			(effects
@@
 			)
 		)
-		(property "Value" "74HCT04"
+		(property "Value" "74ACT04"
 			(at 247.65 121.92 0)
 			(effects
@@
 			)
 		)
-		(property "Value" "2.2k"
+		(property "Value" "1k"
 			(at 119.38 114.3 90)
 			(effects

Commit message: Fix rotated transistor in dupico pal pod
Connections:
- net VCC: now also Q1.1 (E); no longer Q1.3 (C)
- net ZIF_40: now also Q1.3 (C); no longer Q1.1 (E)
Other:
- moved on the sheet: Q1
Changed lines of the file:
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@@
 	(symbol
 		(lib_id "Transistor_BJT:2N3906")
-		(at 106.68 116.84 0)
-		(mirror y)
+		(at 106.68 116.84 180)
 		(unit 1)
 		(exclude_from_sim no)
@@
 		(on_board yes)
 		(dnp no)
-		(fields_autoplaced yes)
 		(property "Reference" "Q1"
-			(at 101.6 115.5699 0)
+			(at 101.6 118.1101 0)
 			(effects
 				(font
@@
 		)
 		(property "Value" "2N3906"
-			(at 101.6 118.1099 0)
+			(at 101.6 115.5701 0)
 			(effects
 				(font
@@
 		)
 		(property "Footprint" "Package_TO_SOT_THT:TO-92_Inline"
-			(at 101.6 118.745 0)
+			(at 101.6 114.935 0)
 			(effects
 				(font
